File: PCB/IO_Block.kicad_sch (KiCad schematic)
At the start: 3 parts

Commit message: Revert "Revert "# Title: Summary, imperative, start upper case, don't end with a period""
This reverts commit 3a20dd9da141c7cb1bae8077342d3450242b15f5.
Parts:
- J? (x3): footprint SHDR10W100P0X500_1X10_5000X900X1250P -> LIB_TB001-500-10BE:SHDR10W100P0X500_1X10_5000X900X1250P
Changed lines of the file:
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@@
       (effects (font (size 1.27 1.27)))
     )
-    (property "Footprint" "SHDR10W100P0X500_1X10_5000X900X1250P" (at 69.85 58.75 0)
+    (property "Footprint" "LIB_TB001-500-10BE:SHDR10W100P0X500_1X10_5000X900X1250P" (at 69.85 58.75 0)
       (effects (font (size 1.27 1.27)) (justify left top) hide)
     )
@@
       (effects (font (size 1.27 1.27)))
     )
-    (property "Footprint" "SHDR10W100P0X500_1X10_5000X900X1250P" (at 69.85 21.92 0)
+    (property "Footprint" "LIB_TB001-500-10BE:SHDR10W100P0X500_1X10_5000X900X1250P" (at 69.85 21.92 0)
       (effects (font (size 1.27 1.27)) (justify left top) hide)
     )
@@
       (effects (font (size 1.27 1.27)))
     )
-    (property "Footprint" "SHDR10W100P0X500_1X10_5000X900X1250P" (at 69.85 -13.64 0)
+    (property "Footprint" "LIB_TB001-500-10BE:SHDR10W100P0X500_1X10_5000X900X1250P" (at 69.85 -13.64 0)
       (effects (font (size 1.27 1.27)) (justify left top) hide)
     )

Commit message: Revert "# Title: Summary, imperative, start upper case, don't end with a period"
This reverts commit 68e2e82ae65b044d3f55e91a7adcee939c25789e.
Parts:
- J? (x3): footprint LIB_TB001-500-10BE:SHDR10W100P0X500_1X10_5000X900X1250P -> SHDR10W100P0X500_1X10_5000X900X1250P
Changed lines of the file:
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@@
       (effects (font (size 1.27 1.27)))
     )
-    (property "Footprint" "LIB_TB001-500-10BE:SHDR10W100P0X500_1X10_5000X900X1250P" (at 69.85 58.75 0)
+    (property "Footprint" "SHDR10W100P0X500_1X10_5000X900X1250P" (at 69.85 58.75 0)
       (effects (font (size 1.27 1.27)) (justify left top) hide)
     )
@@
       (effects (font (size 1.27 1.27)))
     )
-    (property "Footprint" "LIB_TB001-500-10BE:SHDR10W100P0X500_1X10_5000X900X1250P" (at 69.85 21.92 0)
+    (property "Footprint" "SHDR10W100P0X500_1X10_5000X900X1250P" (at 69.85 21.92 0)
       (effects (font (size 1.27 1.27)) (justify left top) hide)
     )
@@
       (effects (font (size 1.27 1.27)))
     )
-    (property "Footprint" "LIB_TB001-500-10BE:SHDR10W100P0X500_1X10_5000X900X1250P" (at 69.85 -13.64 0)
+    (property "Footprint" "SHDR10W100P0X500_1X10_5000X900X1250P" (at 69.85 -13.64 0)
       (effects (font (size 1.27 1.27)) (justify left top) hide)
     )
