File: PCB/IO_Block.kicad_sch (KiCad schematic)
At the start: 3 parts

Commit message: Redesigned, to utilize the ESP32 as the basis
* Implemented EEPROM
* Implemented RTC
* Implemented RS232 and 485
* Implemented CANBus
* Implemented everything
Other:
- company: (none) -> UPB - FIIR - Roboți și sisteme de producție
Changed lines of the file:
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@@
 (kicad_sch (version 20230121) (generator eeschema)
   (paper "A4")
+  (title_block
+    (date "2023-04-23")
+    (rev "1")
+    (company "UPB - FIIR - Roboți și sisteme de producție")
+    (comment 1 "Alexandru-Ioan Anastasiu")
+  )
   (hierarchical_label "GPO_1" (shape output) (at 86.36 99.06 0) (fields_autoplaced)
     (effects (font (size 1.27 1.27)) (justify left))
