File: PCB/IO_Block_1.kicad_sch (KiCad schematic)
At the start: 12 parts, among them IC1 TLP172AM_TPR,E, IC2 TLP172AM_TPR,E, IC3 TLP172AM_TPR,E, IC4 TLP172AM_TPR,E, IC5 TLP172AM_TPR,E, IC6 TLP172AM_TPR,E

Commit message: Revert "Revert "# Title: Summary, imperative, start upper case, don't end with a period""
This reverts commit 3a20dd9da141c7cb1bae8077342d3450242b15f5.
Parts:
- IC1, IC2, IC3, IC4, IC5, IC6: footprint SOIC127P700X230-6N -> LIB_TLP172AM_TPR,E:SOIC127P700X230-6N

Commit message: Revert "# Title: Summary, imperative, start upper case, don't end with a period"
This reverts commit 68e2e82ae65b044d3f55e91a7adcee939c25789e.
Parts:
- IC1, IC2, IC3, IC4, IC5, IC6: footprint LIB_TLP172AM_TPR,E:SOIC127P700X230-6N -> SOIC127P700X230-6N
