File: PCB/PLC-CIM.kicad_sch (KiCad schematic)
At the start: 3 parts, among them IC31 TXS0102DCUTG4, U1 ESP32-DEVKITC

Commit message: Revert "# Title: Summary, imperative, start upper case, don't end with a period"
This reverts commit 68e2e82ae65b044d3f55e91a7adcee939c25789e.
Parts:
- IC31: footprint TXS0102DCUTG4:SOP50P310X90-8N -> SOP50P310X90-8N
Changed lines of the file:
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@@
       (effects (font (size 1.27 1.27)))
     )
-    (property "Footprint" "TXS0102DCUTG4:SOP50P310X90-8N" (at 222.25 237.795 0)
+    (property "Footprint" "SOP50P310X90-8N" (at 222.25 237.795 0)
       (effects (font (size 1.27 1.27)) (justify left top) hide)
     )
