File: PCB/PM.kicad_sch (KiCad schematic)
At the start: 4 parts, among them J4 TC0203620000G, J5 TC0203620000G, J6 TC0203620000G, J7 TC0203620000G

Commit message: Revert "Revert "# Title: Summary, imperative, start upper case, don't end with a period""
This reverts commit 3a20dd9da141c7cb1bae8077342d3450242b15f5.
Parts:
- J4, J5, J6, J7: footprint TC0203620000G -> TC0203620000G:TC0203620000G
Changed lines of the file:
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@@
       (effects (font (size 1.27 1.27)) (justify left))
     )
-    (property "Footprint" "TC0203620000G" (at 184.15 209.855 0)
+    (property "Footprint" "TC0203620000G:TC0203620000G" (at 184.15 209.855 0)
       (effects (font (size 1.27 1.27)) (justify left top) hide)
     )
@@
       (effects (font (size 1.27 1.27)) (justify left))
     )
-    (property "Footprint" "TC0203620000G" (at 184.15 196.52 0)
+    (property "Footprint" "TC0203620000G:TC0203620000G" (at 184.15 196.52 0)
       (effects (font (size 1.27 1.27)) (justify left top) hide)
     )
@@
       (effects (font (size 1.27 1.27)) (justify left))
     )
-    (property "Footprint" "TC0203620000G" (at 139.7 196.52 0)
+    (property "Footprint" "TC0203620000G:TC0203620000G" (at 139.7 196.52 0)
       (effects (font (size 1.27 1.27)) (justify left top) hide)
     )
@@
       (effects (font (size 1.27 1.27)) (justify left))
     )
-    (property "Footprint" "TC0203620000G" (at 139.7 211.76 0)
+    (property "Footprint" "TC0203620000G:TC0203620000G" (at 139.7 211.76 0)
       (effects (font (size 1.27 1.27)) (justify left top) hide)
     )

Commit message: Revert "# Title: Summary, imperative, start upper case, don't end with a period"
This reverts commit 68e2e82ae65b044d3f55e91a7adcee939c25789e.
Parts:
- J4, J5, J6, J7: footprint TC0203620000G:TC0203620000G -> TC0203620000G
Changed lines of the file:
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@@
       (effects (font (size 1.27 1.27)) (justify left))
     )
-    (property "Footprint" "TC0203620000G:TC0203620000G" (at 184.15 209.855 0)
+    (property "Footprint" "TC0203620000G" (at 184.15 209.855 0)
       (effects (font (size 1.27 1.27)) (justify left top) hide)
     )
@@
       (effects (font (size 1.27 1.27)) (justify left))
     )
-    (property "Footprint" "TC0203620000G:TC0203620000G" (at 184.15 196.52 0)
+    (property "Footprint" "TC0203620000G" (at 184.15 196.52 0)
       (effects (font (size 1.27 1.27)) (justify left top) hide)
     )
@@
       (effects (font (size 1.27 1.27)) (justify left))
     )
-    (property "Footprint" "TC0203620000G:TC0203620000G" (at 139.7 196.52 0)
+    (property "Footprint" "TC0203620000G" (at 139.7 196.52 0)
       (effects (font (size 1.27 1.27)) (justify left top) hide)
     )
@@
       (effects (font (size 1.27 1.27)) (justify left))
     )
-    (property "Footprint" "TC0203620000G:TC0203620000G" (at 139.7 211.76 0)
+    (property "Footprint" "TC0203620000G" (at 139.7 211.76 0)
       (effects (font (size 1.27 1.27)) (justify left top) hide)
     )
