File: PCB/RS485.kicad_sch (KiCad schematic)
At the start: 6 parts, among them IC47 SN65HVD75DR, J10 Conn_02x01, J9 Conn_02x01

Commit message: Implemented Output block in PCB Started implementation of Input block in PCB
Parts:
- J10, J9: footprint Connector_PinHeader_2.54mm:PinHeader_2x01_P2.54mm_Horizontal -> Connector_PinHeader_2.54mm:PinHeader_2x01_P2.54mm_Vertical
Changed lines of the file:
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@@
       (effects (font (size 1.27 1.27)) (justify right))
     )
-    (property "Footprint" "Connector_PinHeader_2.54mm:PinHeader_2x01_P2.54mm_Horizontal" (at 222.25 86.36 0)
+    (property "Footprint" "Connector_PinHeader_2.54mm:PinHeader_2x01_P2.54mm_Vertical" (at 222.25 86.36 0)
       (effects (font (size 1.27 1.27)) hide)
     )
@@
       (effects (font (size 1.27 1.27)))
     )
-    (property "Footprint" "Connector_PinHeader_2.54mm:PinHeader_2x01_P2.54mm_Horizontal" (at 177.165 95.25 0)
+    (property "Footprint" "Connector_PinHeader_2.54mm:PinHeader_2x01_P2.54mm_Vertical" (at 177.165 95.25 0)
       (effects (font (size 1.27 1.27)) hide)
     )
@@
       (effects (font (size 1.27 1.27)))
     )
-    (property "Footprint" "Connector_PinHeader_2.54mm:PinHeader_2x01_P2.54mm_Horizontal" (at 177.165 104.775 0)
+    (property "Footprint" "Connector_PinHeader_2.54mm:PinHeader_2x01_P2.54mm_Vertical" (at 177.165 104.775 0)
       (effects (font (size 1.27 1.27)) hide)
     )
@@
       (effects (font (size 1.27 1.27)) (justify right))
     )
-    (property "Footprint" "Connector_PinHeader_2.54mm:PinHeader_2x01_P2.54mm_Horizontal" (at 229.235 86.36 0)
-      (effects (font (size 1.27 1.27)) hide)
-    )
+    (property "Footprint" "Connector_PinHeader_2.54mm:PinHeader_2x01_P2.54mm_Vertical" (at 229.235 86.36 0)
+      (effects (font (size 1.27 1.27)) hide)
+    )
