File: PCB/RTC.kicad_sch (KiCad schematic)
At the start: 1 part

Commit message: Implemented Output block in PCB Started implementation of Input block in PCB
Parts:
- J?: footprint Connector_PinHeader_2.54mm:PinHeader_2x05_P2.54mm_Horizontal -> Connector_PinSocket_2.54mm:PinSocket_2x05_P2.54mm_Vertical
Changed lines of the file:
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@@
       (effects (font (size 1.27 1.27)))
     )
-    (property "Footprint" "Connector_PinHeader_2.54mm:PinHeader_2x05_P2.54mm_Horizontal" (at 186.69 95.885 0)
+    (property "Footprint" "Connector_PinSocket_2.54mm:PinSocket_2x05_P2.54mm_Vertical" (at 186.69 95.885 0)
       (effects (font (size 1.27 1.27)) hide)
     )
