File: PCB/EEPROM.kicad_sch (KiCad schematic)
At the start: 1 part, among them U2 AT24CM02-SSHM-B

Commit message: Implemented Output block in PCB Started implementation of Input block in PCB
Parts:
- U2: footprint SOIC127P600X175-8N -> AT24CM02-SSHM-B:SOIC127P600X175-8N
Changed lines of the file:
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@@
       (effects (font (size 1.27 1.27)))
     )
-    (property "Footprint" "SOIC127P600X175-8N" (at 165.1 193.345 0)
+    (property "Footprint" "AT24CM02-SSHM-B:SOIC127P600X175-8N" (at 165.1 193.345 0)
       (effects (font (size 1.27 1.27)) (justify left top) hide)
     )
