File: PCB/PLC-CIM.kicad_pcb (KiCad board)
At the start: 4 copper layers, 152.7 x 98.9 mm, 124 parts, among them IC1 TLP172AM_TPR,E, IC10 TLV9351IDCKR, IC11 TLV9351IDCKR, IC12 TLV9351IDCKR, IC13 TLP172AM_TPR,E, IC14 TLP172AM_TPR,E, IC15 TLP172AM_TPR,E, IC16 TLP172AM_TPR,E, IC17 TLP172AM_TPR,E, IC18 TLP172AM_TPR,E, IC19 TLV9351IDCKR, IC2 TLP172AM_TPR,E, IC20 TLV9351IDCKR, IC21 TLV9351IDCKR, IC22 TLV9351IDCKR, IC23 TLV9351IDCKR, IC24 TLV9351IDCKR, IC25 TLP172AM_TPR,E, IC26 TLP172AM_TPR,E, IC27 TLP172AM_TPR,E, IC28 TLP172AM_TPR,E, IC29 TLP172AM_TPR,E, IC3 TLP172AM_TPR,E, IC30 TLP172AM_TPR,E, IC31 MAX3221IDBRE4, IC32 TLP172AM_TPR,E, IC33 TLP172AM_TPR,E, IC34 TLP172AM_TPR,E, IC35 TLP172AM_TPR,E, IC36 TLP172AM_TPR,E, IC37 TLP172AM_TPR,E, IC38 TLP172AM_TPR,E, IC39 TLP172AM_TPR,E, IC4 TLP172AM_TPR,E, IC40 TLP172AM_TPR,E, IC41 TLP172AM_TPR,E, IC42 TLP172AM_TPR,E, IC43 TLP172AM_TPR,E, IC44 PCA9555PW,118, IC45 TCAN337DCNR, IC46 PCA9555PW,118, IC47 SN65HVD75DR, IC5 TLP172AM_TPR,E, IC6 TLP172AM_TPR,E, IC7 TLV9351IDCKR, IC8 TLV9351IDCKR, IC9 TLV9351IDCKR, J1 TB001-500-10BE, J10 Conn_02x01, J11 Conn_02x05_Odd_Even, J12 TC0203620000G, J13 750678-1, J14 Conn_02x01, J15 Conn_02x01, J16 Conn_02x01, J17 Conn_02x01, J2 TB001-500-10BE, J3 TB001-500-10BE, J4 TC0203620000G, J5 TC0203620000G, J6 TC0203620000G, J7 TC0203620000G, J8 750678-1, J9 Conn_02x01, U1 ESP32-DEVKITC, U2 AT24CM02-SSHM-B

Commit message: Finalized PCB
Parts:
- added G***: LOGO, LOGO, F.Cu at (147.1, 70.4)
- added G***: LOGO, LOGO, F.Cu at (135.5, 70.5)
- added G***: LOGO, LOGO, F.Cu at (160.5, 68.5)
- added G***: LOGO, LOGO, F.Cu at (147.5, 80.7)
- C1, C2, C3, C4, IC31, IC45, IC47, U2: moved to B.Cu
- moved J16 331.4 mm to (220.7, 84.6)
- moved J14 325.1 mm to (214.5, 86.5), turned to 180 degrees
- moved J17 319.3 mm to (208.6, 94.4), turned to 90 degrees
- moved J15 319.3 mm to (208.6, 86.6), turned to -90 degrees
- moved J4 309.5 mm to (160.9, 61.1), turned to 180 degrees
- moved J5 308.4 mm to (161.6, 79.4), turned to 180 degrees
- moved IC47 304.7 mm to (211.9, 80.3), turned to -90 degrees
- moved J6 304.0 mm to (149.4, 61.1), turned to 180 degrees
- moved J7 296.5 mm to (137.8, 61.1), turned to 180 degrees
- moved J12 272.1 mm to (220.3, 79.6), turned to 90 degrees
- moved IC45 268.9 mm to (211.7, 74.7)
- moved U2 237.1 mm to (117.9, 66.3), turned to 90 degrees
- moved J11 193.6 mm to (129.5, 76.7), turned to 90 degrees
- moved C4 170.9 mm to (96.5, 93.5), turned to 45 degrees
- moved C3 170.4 mm to (96.1, 99.2), turned to 90 degrees
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Connections:
- R10 pad 1: /I Block 1/I_ACT_5 -> MCU_IN_8
- R11 pad 1: /I Block 1/I_ACT_4 -> MCU_IN_9
- R12 pad 1: /I Block 1/I_ACT_3 -> MCU_IN_10
- R13 pad 2: /I Block 1/I_ACT_2 -> MCU_IN_11
- R14 pad 2: /I Block 1/I_ACT_1 -> MCU_IN_12
- R15 pad 2: /I Block 1/I_ACT_6 -> MCU_IN_7
- R16 pad 2: /I Block 1/I_ACT_5 -> MCU_IN_8
- R17 pad 2: /I Block 1/I_ACT_4 -> MCU_IN_9
- R18 pad 2: /I Block 1/I_ACT_3 -> MCU_IN_10
- R25 pad 1: /I Block 2/I_ACT_2 -> MCU_IN_5
- R26 pad 1: /I Block 2/I_ACT_1 -> MCU_IN_6
- R27 pad 1: /I Block 2/I_ACT_6 -> MCU_IN_1
- R28 pad 1: /I Block 2/I_ACT_5 -> MCU_IN_2
- R29 pad 1: /I Block 2/I_ACT_4 -> MCU_IN_3
- R30 pad 1: /I Block 2/I_ACT_3 -> MCU_IN_4
- R31 pad 2: /I Block 2/I_ACT_2 -> MCU_IN_5
- R32 pad 2: /I Block 2/I_ACT_1 -> MCU_IN_6
- R33 pad 2: /I Block 2/I_ACT_6 -> MCU_IN_1
- R34 pad 2: /I Block 2/I_ACT_5 -> MCU_IN_2
- R35 pad 2: /I Block 2/I_ACT_4 -> MCU_IN_3
- R36 pad 2: /I Block 2/I_ACT_3 -> MCU_IN_4
- R7 pad 1: /I Block 1/I_ACT_2 -> MCU_IN_11
- R8 pad 1: /I Block 1/I_ACT_1 -> MCU_IN_12
- R9 pad 1: /I Block 1/I_ACT_6 -> MCU_IN_7
- U1 pad 10: /I Block 2/I_ACT_2 -> MCU_IN_8
- U1 pad 11: /I Block 2/I_ACT_3 -> MCU_IN_9
- U1 pad 12: /I Block 2/I_ACT_4 -> MCU_IN_10
- U1 pad 13: /I Block 2/I_ACT_5 -> MCU_IN_11
- U1 pad 15: /I Block 2/I_ACT_6 -> MCU_IN_12
- U1 pad 3: /I Block 1/I_ACT_1 -> MCU_IN_2
- U1 pad 4: /I Block 1/I_ACT_2 -> MCU_IN_1
- U1 pad 5: /I Block 1/I_ACT_3 -> MCU_IN_7
- U1 pad 6: /I Block 1/I_ACT_4 -> MCU_IN_6
- U1 pad 7: /I Block 1/I_ACT_5 -> MCU_IN_5
- U1 pad 8: /I Block 1/I_ACT_6 -> MCU_IN_4
- U1 pad 9: /I Block 2/I_ACT_1 -> MCU_IN_3
Routing:
- net +3.3V: track 0.00 -> 263.2 mm, vias 0 -> 5
- net +24V: track 298.2 -> 535.2 mm, vias 30 -> 37
- net SDA: track 0.00 -> 212.6 mm, vias 0 -> 1
- net SCL: track 0.00 -> 195.0 mm, vias 0 -> 1
- net GPIO_11: track 29.5 -> 201.0 mm
- net GPIO_12: track 26.3 -> 188.0 mm
- net CAN_RX: track 0.00 -> 136.2 mm, vias 0 -> 1
- net CAN_TX: track 0.00 -> 135.9 mm, vias 0 -> 1
- net MCU_IN_2: track 0.00 -> 134.4 mm
- net CAN_FAULT: track 0.00 -> 133.4 mm, vias 0 -> 1
- net MCU_IN_8: track 0.00 -> 130.2 mm
- net MCU_IN_1: track 0.00 -> 129.1 mm
- net MCU_IN_9: track 0.00 -> 124.2 mm
- net MCU_IN_7: track 0.00 -> 123.8 mm
- net TX1: track 0.00 -> 122.9 mm, vias 0 -> 1
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- added copper zone on B.Cu, net GND
- added copper zone on F.Cu, net GND
- added copper zone on In2.Cu, net GND
Other:
- board size 152.7 x 98.9 mm -> 153.5 x 73.7 mm
- board text added: "If you can read this, please replace your ESP32"
